Commit message: so_arm_100_description: make Gazebo and MoveIt configs compatible
Gazebo
- Remove suffix from libgz-physics-ode-plugin.so
- The .so suffix prevents the library loading on macOS.

Consolidate urdf files
- Add separate xacro files for gazebo and ros2_control
- Add Gazebo xacro file to hold Gazebo plugins and controllers.
- Add ros2_control xacro file to hold controller configuration.
- Add urdf.xacro files for the arm
- Use xacro for robot description.
- Remove unreferenced urdf file so_arm_100.urdf
- Use revolute joints and add limits

Use xacro for robot model
- Remove urdf file replaced by xacro
- so_arm_100_5dof.urdf now replaced by xacro version in launch files.
- Generate so_arm_100_5dof_hardware.urdf from xacro.

Changes to robot model
- Use package:// instead of file:// in urdf
- Add collision to the end effector
- Correct joint limits
- Add joint damping
- Change material to bright yellow.

Update joint_state_pub_gui launch
- Rename file.
- Update package paths.
- Use xacro.
- Remove unused imports

Correct joint axis orientation and offsets
- Move joint state gui launch and rviz config.
- Add prefix launch argument.
- Allow either gz_ros2_control or topic based control to be selected in gazebo.xacro.
- Add param use_topic_hardware_interface
- Add param ros2_controllers_file
- Add parameter ros2_controllers_file to gazebo xacro.
- Resolve cyclic dependency issue (config is in moveit_config -> description).

Signed-off-by: Rhys Mainwaring <rhys.mainwaring@me.com>

File: so_arm_100_description/urdf/so_arm_100_5dof_arm.urdf.xacro (robot description, xacro)
@@ -1,27 +1,28 @@
 <?xml version="1.0" encoding="utf-8"?>
-<!-- This URDF was automatically created by SolidWorks to URDF Exporter! Originally created by Stephen Brawner (brawner@gmail.com)
-     Commit Version: 1.6.0-1-g15f4949  Build Version: 1.6.7594.29634
-     For more information, please see http://wiki.ros.org/sw_urdf_exporter -->
-<robot
-  name="so_arm_100">
-  <!-- <link name="world"/>
-  <joint name="world_to_base" type="fixed">
-    <parent link="world"/>
-    <child link="base_link"/>
-    <origin xyz="0 0 0" rpy="0 0 0"/>
-  </joint> -->
-  <link
-    name="base_link">
+<!--
+Modified from auto-generated original:
+- Add xacro macros and properties.
+- Add end effector
+This URDF was automatically created by SolidWorks to URDF Exporter!
+Originally created by Stephen Brawner (brawner@gmail.com)
+Commit Version: 1.6.0-1-g15f4949  Build Version: 1.6.7594.29634
+For more information, please see http://wiki.ros.org/sw_urdf_exporter
+-->
+<robot xmlns:xacro="http://www.ros.org/wiki/xacro">
+  <xacro:macro name="so_arm_100_5dof" params="prefix=''">
+  <xacro:property
+    name="meshes_file_directory"
+    value="package://so_arm_100_description/models/so_arm_100_5dof/meshes"/>
+  <link name="${prefix}base_link">
     <gazebo>
       <material>Gazebo/Grey</material>
     </gazebo>
   </link>
-  <joint name="base_link_joint" type="fixed">
-    <parent link="base_link"/>
-    <child link="Base"/>
+  <joint name="${prefix}base_link_joint" type="fixed">
+    <parent link="${prefix}base_link"/>
+    <child link="${prefix}Base"/>
     <origin xyz="0 0 0" rpy="0 0 0"/>
   </joint>
-  <link
-    name="Base">
+  <link name="${prefix}Base">
     <inertial>
       <origin
@@ -44,24 +45,21 @@
       <geometry>
         <mesh
-          filename="package://so_arm_100_moveit_config/models/so_arm_100_5dof/meshes/Base.STL" />
-      </geometry>
-      <material
-        name="">
-        <color
-          rgba="0.792156862745098 0.819607843137255 0.933333333333333 1" />
-      </material>
-    </visual>
-    <collision>
-      <origin
-        xyz="0 0 0"
-        rpy="0 0 0" />
-      <geometry>
-        <mesh
-          filename="package://so_arm_100_moveit_config/models/so_arm_100_5dof/meshes/Base.STL" />
-      </geometry>
-    </collision>
-  </link>
-  <link
-    name="Shoulder_Rotation_Pitch">
+          filename="${meshes_file_directory}/Base.STL" />
+      </geometry>
+      <material name="brightyellow" >
+        <color rgba="1.0 0.9921568627450981 0.00392156862745098 1.0" />
+      </material>
+    </visual>
+    <collision>
+      <origin
+        xyz="0 0 0"
+        rpy="0 0 0" />
+      <geometry>
+        <mesh
+          filename="${meshes_file_directory}/Base.STL" />
+      </geometry>
+    </collision>
+  </link>
+  <link name="${prefix}Shoulder_Rotation_Pitch">
     <inertial>
       <origin
@@ -84,37 +82,34 @@
       <geometry>
         <mesh
-          filename="package://so_arm_100_moveit_config/models/so_arm_100_5dof/meshes/Shoulder_Rotation_Pitch.STL" />
-      </geometry>
-      <material
-        name="">
-        <color
-          rgba="0.792156862745098 0.819607843137255 0.933333333333333 1" />
-      </material>
-    </visual>
-    <collision>
-      <origin
-        xyz="0 0 0"
-        rpy="0 0 0" />
-      <geometry>
-        <mesh
-          filename="package://so_arm_100_moveit_config/models/so_arm_100_5dof/meshes/Shoulder_Rotation_Pitch.STL" />
-      </geometry>
-    </collision>
-  </link>
-  <joint
-    name="Shoulder_Rotation"
-    type="continuous">
+          filename="${meshes_file_directory}/Shoulder_Rotation_Pitch.STL" />
+      </geometry>
+      <material name="brightyellow" >
+        <color rgba="1.0 0.9921568627450981 0.00392156862745098 1.0" />
+      </material>
+    </visual>
+    <collision>
+      <origin
+        xyz="0 0 0"
+        rpy="0 0 0" />
+      <geometry>
+        <mesh
+          filename="${meshes_file_directory}/Shoulder_Rotation_Pitch.STL" />
+      </geometry>
+    </collision>
+  </link>
+  <joint name="${prefix}Shoulder_Rotation" type="revolute">
     <origin
       xyz="0 -0.0452 0.0165"
       rpy="1.5708 0 0" />
     <parent
-      link="Base" />
-    <child
-      link="Shoulder_Rotation_Pitch" />
-    <axis
-      xyz="0 1 0" />
-  </joint>
-  <link
-    name="Upper_Arm">
+      link="${prefix}Base" />
+    <child
+      link="${prefix}Shoulder_Rotation_Pitch" />
+    <axis
+      xyz="0 -1 0" />
+    <limit effort="1000" lower="-1.96" upper="1.96" velocity="5.0"/>
+    <dynamics damping="0.1"/>
+  </joint>
+  <link name="${prefix}Upper_Arm">
     <inertial>
       <origin
@@ -137,37 +132,34 @@
       <geometry>
         <mesh
-          filename="package://so_arm_100_moveit_config/models/so_arm_100_5dof/meshes/Upper_Arm.STL" />
-      </geometry>
-      <material
-        name="">
-        <color
-          rgba="0.792156862745098 0.819607843137255 0.933333333333333 1" />
-      </material>
-    </visual>
-    <collision>
-      <origin
-        xyz="0 0 0"
-        rpy="0 0 0" />
-      <geometry>
-        <mesh
-          filename="package://so_arm_100_moveit_config/models/so_arm_100_5dof/meshes/Upper_Arm.STL" />
-      </geometry>
-    </collision>
-  </link>
-  <joint
-    name="Shoulder_Pitch"
-    type="continuous">
+          filename="${meshes_file_directory}/Upper_Arm.STL" />
+      </geometry>
+      <material name="brightyellow" >
+        <color rgba="1.0 0.9921568627450981 0.00392156862745098 1.0" />
+      </material>
+    </visual>
+    <collision>
+      <origin
+        xyz="0 0 0"
+        rpy="0 0 0" />
+      <geometry>
+        <mesh
+          filename="${meshes_file_directory}/Upper_Arm.STL" />
+      </geometry>
+    </collision>
+  </link>
+  <joint name="${prefix}Shoulder_Pitch" type="revolute">
     <origin
       xyz="0 0.1025 0.0306"
       rpy="0 0 0" />
     <parent
-      link="Shoulder_Rotation_Pitch" />
-    <child
-      link="Upper_Arm" />
+      link="${prefix}Shoulder_Rotation_Pitch" />
+    <child
+      link="${prefix}Upper_Arm" />
     <axis
       xyz="1 0 0" />
-  </joint>
-  <link
-    name="Lower_Arm">
+    <limit effort="1000" lower="-1.745" upper="1.745" velocity="5.0"/>
+    <dynamics damping="0.1"/>
+  </joint>
+  <link name="${prefix}Lower_Arm">
     <inertial>
       <origin
@@ -190,37 +182,34 @@
       <geometry>
         <mesh
-          filename="package://so_arm_100_moveit_config/models/so_arm_100_5dof/meshes/Lower_Arm.STL" />
-      </geometry>
-      <material
-        name="">
-        <color
-          rgba="0.792156862745098 0.819607843137255 0.933333333333333 1" />
-      </material>
-    </visual>
-    <collision>
-      <origin
-        xyz="0 0 0"
-        rpy="0 0 0" />
-      <geometry>
-        <mesh
-          filename="package://so_arm_100_moveit_config/models/so_arm_100_5dof/meshes/Lower_Arm.STL" />
-      </geometry>
-    </collision>
-  </link>
-  <joint
-    name="Elbow"
-    type="continuous">
+          filename="${meshes_file_directory}/Lower_Arm.STL" />
+      </geometry>
+      <material name="brightyellow" >
+        <color rgba="1.0 0.9921568627450981 0.00392156862745098 1.0" />
+      </material>
+    </visual>
+    <collision>
+      <origin
+        xyz="0 0 0"
+        rpy="0 0 0" />
+      <geometry>
+        <mesh
+          filename="${meshes_file_directory}/Lower_Arm.STL" />
+      </geometry>
+    </collision>
+  </link>
+  <joint name="${prefix}Elbow" type="revolute">
     <origin
       xyz="0 0.11257 0.028"
       rpy="0 0 0" />
     <parent
-      link="Upper_Arm" />
-    <child
-      link="Lower_Arm" />
+      link="${prefix}Upper_Arm" />
+    <child
+      link="${prefix}Lower_Arm" />
     <axis
       xyz="1 0 0" />
-  </joint>
-  <link
-    name="Wrist_Pitch_Roll">
+    <limit effort="1000" lower="-1.5" upper="1.5" velocity="5.0"/>
+    <dynamics damping="0.1"/>
+  </joint>
+  <link name="${prefix}Wrist_Pitch_Roll">
     <inertial>
       <origin
@@ -243,37 +232,34 @@
       <geometry>
         <mesh
-          filename="package://so_arm_100_moveit_config/models/so_arm_100_5dof/meshes/Wrist_Pitch_Roll.STL" />
-      </geometry>
-      <material
-        name="">
-        <color
-          rgba="0.792156862745098 0.819607843137255 0.933333333333333 1" />
-      </material>
-    </visual>
-    <collision>
-      <origin
-        xyz="0 0 0"
-        rpy="0 0 0" />
-      <geometry>
-        <mesh
-          filename="package://so_arm_100_moveit_config/models/so_arm_100_5dof/meshes/Wrist_Pitch_Roll.STL" />
-      </geometry>
-    </collision>
-  </link>
-  <joint
-    name="Wrist_Pitch"
-    type="continuous">
+          filename="${meshes_file_directory}/Wrist_Pitch_Roll.STL" />
+      </geometry>
+      <material name="brightyellow" >
+        <color rgba="1.0 0.9921568627450981 0.00392156862745098 1.0" />
+      </material>
+    </visual>
+    <collision>
+      <origin
+        xyz="0 0 0"
+        rpy="0 0 0" />
+      <geometry>
+        <mesh
+          filename="${meshes_file_directory}/Wrist_Pitch_Roll.STL" />
+      </geometry>
+    </collision>
+  </link>
+  <joint name="${prefix}Wrist_Pitch" type="revolute">
     <origin
       xyz="0 0.0052 0.1349"
-      rpy="0 0 0" />
-    <parent
-      link="Lower_Arm" />
-    <child
-      link="Wrist_Pitch_Roll" />
+      rpy="-1.57079 0 0" />
+    <parent
+      link="${prefix}Lower_Arm" />
+    <child
+      link="${prefix}Wrist_Pitch_Roll" />
     <axis
       xyz="1 0 0" />
-  </joint>
-  <link
-    name="Fixed_Gripper">
+    <limit effort="1000" lower="-1.658" upper="1.658" velocity="5.0"/>
+    <dynamics damping="0.1"/>
+  </joint>
+  <link name="${prefix}Fixed_Gripper">
     <inertial>
       <origin
@@ -296,37 +282,34 @@
       <geometry>
         <mesh
-          filename="package://so_arm_100_moveit_config/models/so_arm_100_5dof/meshes/Fixed_Gripper.STL" />
-      </geometry>
-      <material
-        name="">
-        <color
-          rgba="0.792156862745098 0.819607843137255 0.933333333333333 1" />
-      </material>
-    </visual>
-    <collision>
-      <origin
-        xyz="0 0 0"
-        rpy="0 0 0" />
-      <geometry>
-        <mesh
-          filename="package://so_arm_100_moveit_config/models/so_arm_100_5dof/meshes/Fixed_Gripper.STL" />
-      </geometry>
-    </collision>
-  </link>
-  <joint
-    name="Wrist_Roll"
-    type="continuous">
+          filename="${meshes_file_directory}/Fixed_Gripper.STL" />
+      </geometry>
+      <material name="brightyellow" >
+        <color rgba="1.0 0.9921568627450981 0.00392156862745098 1.0" />
+      </material>
+    </visual>
+    <collision>
+      <origin
+        xyz="0 0 0"
+        rpy="0 0 0" />
+      <geometry>
+        <mesh
+          filename="${meshes_file_directory}/Fixed_Gripper.STL" />
+      </geometry>
+    </collision>
+  </link>
+  <joint name="${prefix}Wrist_Roll" type="revolute">
     <origin
       xyz="0 -0.0601 0"
-      rpy="0 0 0" />
-    <parent
-      link="Wrist_Pitch_Roll" />
-    <child
-      link="Fixed_Gripper" />
+      rpy="0 1.57079 0" />
+    <parent
+      link="${prefix}Wrist_Pitch_Roll" />
+    <child
+      link="${prefix}Fixed_Gripper" />
     <axis
       xyz="0 1 0" />
-  </joint>
-  <link
-    name="Moving_Jaw">
+    <limit effort="1000" lower="-2.75" upper="2.75" velocity="5.0"/>
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