Commit message: so_arm_100_moveit_config: make Gazebo and MoveIt configs compatible
Update references in so_arm_100.urdf.xacro

Update configs
- Enable velocity state interface for gripper.
- Ensure initial positions are floats.
- Set additional parameters on the so_arm_100_controller/SOARM100Interface
- Reduce controller rate from 1000 Hz to 100 Hz
- Update joint limits
- Add newline at end of file
- Update kinematics config
- Update .setup_assistant

Edit srdf config
- Update srdf group states, virtual joint and collisions.

Standardise controller names for moveit and ros2_control
- Update moveit rviz config
- Rename controllers.yaml to hardware_controllers.yaml to clarify purpose.

Update launch scripts
- STS3215 servos support speed and load feedback
- Depends on updated so_arm_100_interface
- Disable position_only_ik
  - (disables the interactive marker rotation controls in riviz)
- Restore the original moveit rviz config
- Rename modified rviz config to moveit.xtra.rviz
- Rename joint_trajectory_controller to arm_controller to be consistent with hardware

Rework moveit launch script
- Follow the approach used in OpenMANIPULATOR-X.
- Restore the demo.launch.py as generated by the setup assistant.

Update controllers
- Use position_controllers/JointGroupPositionController for gripper
- Use consistent controller naming
- Use name arm_controller for joint_trajectory_controller/JointTrajectoryController
- Use name gripper_controller for position_controllers/JointGroupPositionController
- Remove velocity state interfaces
- Correct gripper joint group states

- Add params to ros2_control xacro
- Add params with defaults for the servo hardware interface.
- Pass servo settings to hardware controller

- Rename end effector joint
- Change gripper_controller type to parallel_gripper_action_controller/GripperActionController
- Enable velocity and effort interfaces for hardware.
- Add arm effort controller to hardware controllers

Signed-off-by: Rhys Mainwaring <rhys.mainwaring@me.com>

File: so_arm_100_moveit_config/config/so_arm_100.ros2_control.xacro (robot description, xacro)
@@ -1,5 +1,5 @@
 <?xml version="1.0"?>
 <robot xmlns:xacro="http://www.ros.org/wiki/xacro">
-    <xacro:macro name="so_arm_100_ros2_control" params="name initial_positions_file use_fake_hardware" >
+    <xacro:macro name="so_arm_100_ros2_control" params="name initial_positions_file use_fake_hardware serial_port:=^|/dev/ttyUSB0 serial_baudrate:=^|1000000 servo_speed:=^|2400 servo_acceleration:=^|50" >
         <xacro:property name="initial_positions" value="${xacro.load_yaml(initial_positions_file)['initial_positions']}"/>
         <ros2_control name="${name}" type="system">
@@ -11,6 +11,8 @@
                     <plugin>so_arm_100_controller/SOARM100Interface</plugin>
                     <param name="use_serial">true</param>
-                    <param name="serial_port">/dev/ttyUSB0</param>
-                    <param name="serial_baudrate">1000000</param>
+                    <param name="serial_port">${serial_port}</param>
+                    <param name="serial_baudrate">${serial_baudrate}</param>
+                    <param name="servo_speed">${servo_speed}</param>
+                    <param name="servo_acceleration">${servo_acceleration}</param>
                 </xacro:unless>
             </hardware>

File: so_arm_100_moveit_config/config/so_arm_100.urdf.xacro (robot description, xacro)
@@ -1,13 +1,21 @@
 <?xml version="1.0"?>
-<robot xmlns:xacro="http://www.ros.org/wiki/xacro" name="so_100_arm">
+<robot xmlns:xacro="http://www.ros.org/wiki/xacro" name="so_arm_100">
     <xacro:arg name="initial_positions_file" default="initial_positions.yaml" />
     <xacro:arg name="use_fake_hardware" default="false"/>
-    <!-- Import so_100_arm urdf file -->
-    <xacro:include filename="$(find so_100_arm)/urdf/so_100_arm_5dof_hardware.urdf" />
+    <xacro:arg name="serial_port" default="/tty/USB0"/>
+    <xacro:arg name="serial_baudrate" default="1000000"/>
+    <xacro:arg name="servo_speed" default="2400"/>
+    <xacro:arg name="servo_acceleration" default="50"/>
+    <!-- Import so_arm_100 urdf file -->
+    <xacro:include filename="$(find so_arm_100_description)/urdf/so_arm_100_5dof_hardware.urdf" />
     <!-- Import control_xacro -->
-    <xacro:include filename="so_100_arm.ros2_control.xacro" />
-    <xacro:so_100_arm_ros2_control
-        name="SO100ARM"
+    <xacro:include filename="so_arm_100.ros2_control.xacro" />
+    <xacro:so_arm_100_ros2_control
+        name="SOARM100"
         initial_positions_file="$(arg initial_positions_file)"
-        use_fake_hardware="$(arg use_fake_hardware)"/>
+        use_fake_hardware="$(arg use_fake_hardware)"
+        serial_port="$(arg serial_port)"
+        serial_baudrate="$(arg serial_baudrate)"
+        servo_speed="$(arg servo_speed)"
+        servo_acceleration="$(arg servo_acceleration)" />
 </robot>

Commit message: so_arm_100_moveit_config: move files to so_arm_100_moveit_config
- Move files to subpackage so_arm_100_moveit_config
- Edit package references.
- Use standard tag for Apache 2.0 license

Signed-off-by: Rhys Mainwaring <rhys.mainwaring@me.com>

File: so_arm_100_moveit_config/config/so_arm_100.ros2_control.xacro (robot description, xacro)
@@ -1,5 +1,5 @@
 <?xml version="1.0"?>
 <robot xmlns:xacro="http://www.ros.org/wiki/xacro">
-    <xacro:macro name="so_100_arm_ros2_control" params="name initial_positions_file use_fake_hardware" >
+    <xacro:macro name="so_arm_100_ros2_control" params="name initial_positions_file use_fake_hardware" >
         <xacro:property name="initial_positions" value="${xacro.load_yaml(initial_positions_file)['initial_positions']}"/>
         <ros2_control name="${name}" type="system">
