Commit message: so_arm_100_description: add option to set initial_positions in Gazebo joint controllers
- Allow optional initial positions file to be passed to Gazebo xacro.

Signed-off-by: Rhys Mainwaring <rhys.mainwaring@me.com>

File: so_arm_100_description/gazebo/so_arm_100_5dof.gazebo.xacro (robot description, xacro)
@@ -1,11 +1,15 @@
 <?xml version="1.0"?>
 <robot xmlns:xacro="http://ros.org/wiki/xacro">
-  <xacro:macro name="so_arm_100_5dof_gazebo" params="prefix ros2_controllers_file:=^|'' use_topic_hardware_interface:=^|false">
+  <xacro:macro name="so_arm_100_5dof_gazebo" params="prefix initial_positions_file:=^|'' ros2_controllers_file:=^|'' use_topic_hardware_interface:=^|false">
   <!--
   Parameters
       prefix: prefix for joints and links
+      initial_positions_file: initial positions file for joints
       ros2_controllers_file: ros2_controller configuration file for gz_ros2_control
       use_topic_hardware_interface: true if using topic based control
   -->
+  <xacro:if value="${initial_positions_file != ''}">
+      <xacro:property name="initial_positions" value="${xacro.load_yaml(initial_positions_file)['initial_positions']}"/>
+  </xacro:if>
   <gazebo>
     <plugin name="gz::sim::systems::JointStatePublisher"
@@ -52,4 +56,7 @@
         <cmd_max>100.0</cmd_max>
         <cmd_min>-100.0</cmd_min>
+        <xacro:if value="${initial_positions_file != ''}">
+          <initial_position>${initial_positions['Shoulder_Rotation']}</initial_position>
+        </xacro:if>
       </plugin>
       <plugin name="gz::sim::systems::JointPositionController"
@@ -64,4 +71,7 @@
         <cmd_max>100.0</cmd_max>
         <cmd_min>-100.0</cmd_min>
+        <xacro:if value="${initial_positions_file != ''}">
+          <initial_position>${initial_positions['Shoulder_Pitch']}</initial_position>
+        </xacro:if>
       </plugin>
       <plugin name="gz::sim::systems::JointPositionController"
@@ -76,4 +86,7 @@
         <cmd_max>100.0</cmd_max>
         <cmd_min>-100.0</cmd_min>
+        <xacro:if value="${initial_positions_file != ''}">
+          <initial_position>${initial_positions['Elbow']}</initial_position>
+        </xacro:if>
       </plugin>
       <plugin name="gz::sim::systems::JointPositionController"
@@ -88,4 +101,7 @@
         <cmd_max>100.0</cmd_max>
         <cmd_min>-100.0</cmd_min>
+        <xacro:if value="${initial_positions_file != ''}">
+          <initial_position>${initial_positions['Wrist_Pitch']}</initial_position>
+        </xacro:if>
       </plugin>
       <plugin name="gz::sim::systems::JointPositionController"
@@ -100,4 +116,7 @@
         <cmd_max>100.0</cmd_max>
         <cmd_min>-100.0</cmd_min>
+        <xacro:if value="${initial_positions_file != ''}">
+          <initial_position>${initial_positions['Wrist_Roll']}</initial_position>
+        </xacro:if>
       </plugin>
       <plugin name="gz::sim::systems::JointPositionController"
@@ -112,4 +131,7 @@
         <cmd_max>100.0</cmd_max>
         <cmd_min>-100.0</cmd_min>
+        <xacro:if value="${initial_positions_file != ''}">
+          <initial_position>${initial_positions['Gripper']}</initial_position>
+        </xacro:if>
       </plugin>
     </xacro:if>

File: so_arm_100_description/urdf/so_arm_100_5dof.urdf.xacro (robot description, xacro)
@@ -2,4 +2,5 @@
 <robot name="so_arm_100_5dof" xmlns:xacro="http://ros.org/wiki/xacro">
   <xacro:arg name="prefix" default="" />
+  <xacro:arg name="initial_positions_file" default="" />
   <xacro:arg name="use_sim" default="false" />
   <xacro:arg name="use_topic_hardware_interface" default="false" />
@@ -22,4 +23,5 @@
       <xacro:so_arm_100_5dof_gazebo
         prefix="$(arg prefix)"
+        initial_positions_file="$(arg initial_positions_file)"
         ros2_controllers_file="$(arg ros2_controllers_file)"
         use_topic_hardware_interface="$(arg use_topic_hardware_interface)" />
